File: schematics/schematic.kicad_sch (KiCad schematic)
At the start: 46 parts, among them J1 Barrel Jack, J2 Conn_01x02_Pin, Q1 2N2222, SW1 SW_SPDT, SW2 SW_SPST, SW3 SW_MEC_5G, SW4 SW_SPST, U2 74LS374, U3 ATF16V8B, U4 LM7805_TO220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

Commit message: forgot this last night
Parts:
- added R8, R9: 330, symbol ESD:R
- added U8: 24LC16, symbol ESD:24LC16
Connections:
- net GND: now also U8.4 (GND)
- net P1.1: now also U1.2 (P1.1/T2EX/SS)
- net VCC: now also R8.1, R9.1
- net P1.4: now reaches U1.5 (P1.4/CEX1)
- net P1.4: now also R8.2, U8.5 (SDA)
- net P1.5: now reaches U1.6 (P1.5/CEX2/MISO)
- net P1.5: now also R9.2, U8.6 (SCL)
- net P1.6: now reaches U1.7 (P1.6/CEX3/SCK)
- net P1.6: now also U8.7 (WP)

Commit message: part 2 done
Parts:
- added U9: ~, symbol ESD:DMC16433
Connections:
- net P1.6 is gone; now on net GND: U1.7 (P1.6/CEX3/SCK), U8.7 (WP)
- net GND: now also U9.1 (VSS), U9.13 (DB6), U9.3 (VEE), U9.4 (RS)
- net P1.1: now also R8.2, U8.5 (SDA), U9.8 (DB1); no longer R6.1
- net P1.4: now also U9.11 (DB4); no longer R8.2, U8.5 (SDA)
- net P1.5: now also U9.12 (DB5), U9.5 (R/W); no longer R9.2, U8.6 (SCL)
- net VCC: now also U8.8 (VCC), U9.2 (VDD)
- net E: now reaches U3.17 (I/O)
- net E: now also U9.6 (E)
- net P1.0: now reaches U1.1 (P1.0/T2)
- net P1.0: now also R9.2, U8.6 (SCL), U9.7 (DB0)
- net P1.2: now reaches U1.3 (P1.2/ECI)
- net P1.2: now also U9.9 (DB2)
- net P1.3: now reaches U1.4 (P1.3CEX0)
- net P1.3: now also U9.10 (DB3)
- net P1.7: now reaches U1.8 (P1.7CEX4/MOSI)
- net P1.7: now also U9.14 (DB7)
